Commit message: 更新仿真资产与文档

File: simulation/sim2sim/assets/cyvet/urdf/cyvet.urdf (robot description, URDF)
Before this commit: robot uni_0417, 17 links, 16 joints
Links:
- link BASE_LINK: mass 7.3003205393524802 -> 7.7; geometry collision box size=0.025 0.0332 0.09; collision box size=0.11 0.106 0.072
- link FL_ABAD_LINK: mass 0.320329944374416 -> 0.12099999999999998; geometry collision cylinder length=0.055 radius=0.04; visual mesh filename=../meshes/fl_abad_link.stl
- link FL_FOOT_LINK: mass 0.0589523342854384 -> 0.07; geometry collision sphere radius=0.023; visual mesh filename=../meshes/fl_foot_link.stl
- link FL_HIP_LINK: mass 1.3300000000000001 -> 1.438; geometry collision box size=0.046 0.03 0.18; visual mesh filename=../meshes/fl_hip_link.stl
- link FL_KNEE_LINK: mass 0.14 -> 0.167; geometry collision box size=0.02 0.02 0.124; collision box size=0.022 0.022 0.075
- link FR_ABAD_LINK: mass 0.320332974895231 -> 0.12100290502215937; geometry collision cylinder length=0.055 radius=0.04; visual mesh filename=../meshes/fr_abad_link.stl
- link FR_FOOT_LINK: mass 0.0589523342854384 -> 0.07; geometry collision sphere radius=0.023; visual mesh filename=../meshes/fr_foot_link.stl
- link FR_HIP_LINK: mass 1.3300000000000001 -> 1.438; geometry collision box size=0.046 0.03 0.18; visual mesh filename=../meshes/fr_hip_link.stl
- link FR_KNEE_LINK: mass 0.14 -> 0.1670130542472294; geometry collision box size=0.02 0.02 0.124; collision box size=0.022 0.022 0.075
- link RL_ABAD_LINK: mass 0.320333006502764 -> 0.12100296460958171; geometry collision cylinder length=0.055 radius=0.04; visual mesh filename=../meshes/rl_abad_link.stl
- link RL_FOOT_LINK: mass 0.0589523342854384 -> 0.07; geometry collision sphere radius=0.023; visual mesh filename=../meshes/rl_foot_link.stl
- link RL_HIP_LINK: mass 1.3300000000000001 -> 1.438; geometry collision box size=0.046 0.03 0.18; visual mesh filename=../meshes/rl_hip_link.stl
- link RL_KNEE_LINK: mass 0.14 -> 0.16700002369296388; geometry collision box size=0.02 0.02 0.124; collision box size=0.022 0.022 0.075
- link RR_ABAD_LINK: mass 0.320330247102786 -> 0.12100045029579216; geometry collision cylinder length=0.055 radius=0.04; visual mesh filename=../meshes/rr_abad_link.stl
- link RR_FOOT_LINK: mass 0.0589523342854384 -> 0.07; geometry collision sphere radius=0.023; visual mesh filename=../meshes/rr_foot_link.stl
- link RR_HIP_LINK: mass 1.3300000000000001 -> 1.438; geometry collision box size=0.046 0.03 0.18; visual mesh filename=../meshes/rr_hip_link.stl
- link RR_KNEE_LINK: mass 0.14 -> 0.16701135121073604; geometry collision box size=0.02 0.02 0.124; collision box size=0.022 0.022 0.075
